File: Amplifier.kicad_sch (KiCad schematic)
At the start: 22 parts, among them U4 TDA1517/N3, U5 TEA2025B

Commit message: Fix BOM Error
Parts:
- CT1, CT2, CT4, CT7, CT8: LCSC C112487 -> C106447
- R16, R17, R19, R20: value 2.7kΩ -> 27kΩ; LCSC C17530 -> C17593
Changed lines of the file:
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@@
 			)
 		)
-		(property "LCSC" "C112487"
+		(property "LCSC" "C106447"
 			(at 49.53 54.61 0)
 			(effects
@@
 			)
 		)
-		(property "LCSC" "C112487"
+		(property "LCSC" "C106447"
 			(at 85.09 71.12 0)
 			(effects
@@
 			)
 		)
-		(property "Value" "2.7kΩ"
-			(at 151.384 67.3099 0)
+		(property "Value" "27kΩ"
+			(at 152.146 67.31 0)
 			(effects
 				(font
@@
 			)
 		)
-		(property "LCSC" "C17530"
+		(property "LCSC" "C17593"
 			(at 158.75 66.04 0)
 			(effects
@@
 			)
 		)
-		(property "LCSC" "C112487"
+		(property "LCSC" "C106447"
 			(at 162.56 48.26 0)
 			(effects
@@
 			)
 		)
-		(property "Value" "2.7kΩ"
+		(property "Value" "27kΩ"
 			(at 66.04 65.024 90)
 			(effects
@@
 			)
 		)
-		(property "LCSC" "C17530"
+		(property "LCSC" "C17593"
 			(at 66.04 59.69 0)
 			(effects
@@
 			)
 		)
-		(property "Value" "2.7kΩ"
+		(property "Value" "27kΩ"
 			(at 165.1 65.278 90)
 			(effects
@@
 			)
 		)
-		(property "LCSC" "C17530"
+		(property "LCSC" "C17593"
 			(at 165.1 59.69 0)
 			(effects
@@
 			)
 		)
-		(property "Value" "2.7kΩ"
-			(at 79.756 67.564 0)
+		(property "Value" "27kΩ"
+			(at 79.248 67.564 0)
 			(effects
 				(font
@@
 			)
 		)
-		(property "LCSC" "C17530"
+		(property "LCSC" "C17593"
 			(at 72.39 66.04 0)
 			(effects
@@
 			)
 		)
-		(property "LCSC" "C112487"
+		(property "LCSC" "C106447"
 			(at 67.31 48.26 0)
 			(effects
@@
 			)
 		)
-		(property "LCSC" "C112487"
+		(property "LCSC" "C106447"
 			(at 181.61 54.61 0)
 			(effects
