File: Audician 32 Plus Replica.kicad_pcb (KiCad board)
At the start: 2 copper layers, 158.4 x 80.7 mm, 190 parts, among them CN1 CD-ROM, CN2 Waveblaster, J1 Bus_ISA_16bit, J10 Conn_01x04, J11 Conn_01x04, J13 Conn_01x04, J2 Audio Out, J3 Line Input, J4 Microphone, J5 Gameport, J7 Conn_01x04, J8 Conn_01x04, J9 Conn_01x04, Q1 HT7251, Q2 MMBT3904, U1 QS1000, U10 74LS138, U2 QS1001A, U3 TDA1311AT, U4 TDA1517/N3, U5 TEA2025B, U6 YMF719E-S, U7 Mysterious Chip, U8 MK1420S, U9 93C66C, X1 24MHz, X2 33.8688MHz, X3 24.576MHz

Commit message: Fix BOM Error
Parts:
- R16, R17, R19, R20: value 2.7kΩ -> 27kΩ
Changed lines of the file:
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@@
 			)
 		)
-		(property "Value" "2.7kΩ"
+		(property "Value" "27kΩ"
 			(at 0 1.65 90)
 			(layer "F.Fab")
@@
 			)
 		)
-		(property "LCSC" "C17530"
+		(property "LCSC" "C17593"
 			(at 0 0 0)
 			(layer "F.SilkS")
@@
 			)
 		)
-		(property "Value" "2.7kΩ"
+		(property "Value" "27kΩ"
 			(at 0 1.65 90)
 			(layer "F.Fab")
@@
 			)
 		)
-		(property "LCSC" "C17530"
+		(property "LCSC" "C17593"
 			(at 0 0 0)
 			(layer "F.SilkS")
@@
 			)
 		)
-		(property "Value" "2.7kΩ"
+		(property "Value" "27kΩ"
 			(at 0 1.65 90)
 			(layer "F.Fab")
@@
 			)
 		)
-		(property "LCSC" "C17530"
+		(property "LCSC" "C17593"
 			(at 0 0 0)
 			(layer "F.SilkS")
@@
 			)
 		)
-		(property "Value" "2.7kΩ"
+		(property "Value" "27kΩ"
 			(at 0 1.65 90)
 			(layer "F.Fab")
@@
 			)
 		)
-		(property "LCSC" "C17530"
+		(property "LCSC" "C17593"
 			(at 0 0 0)
 			(layer "F.SilkS")

Commit message: Update BOM
Parts:
- C38, C39: value 22pF -> 4pF
Changed lines of the file:
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@@
 			)
 		)
-		(property "Value" "22pF"
+		(property "Value" "4pF"
 			(at 0 1.68 90)
 			(layer "F.Fab")
@@
 			)
 		)
-		(property "LCSC" "C1804"
+		(property "LCSC" "C1819"
 			(at 0 0 0)
 			(layer "F.SilkS")
@@
 			)
 		)
-		(property "LCSC" "C17514"
+		(property "LCSC" "C17614"
 			(at 0 0 0)
 			(layer "F.SilkS")
@@
 			)
 		)
-		(property "Value" "22pF"
+		(property "Value" "4pF"
 			(at 0 1.68 90)
 			(layer "F.Fab")
@@
 			)
 		)
-		(property "LCSC" "C1804"
+		(property "LCSC" "C1819"
 			(at 0 0 0)
 			(layer "F.SilkS")

Commit message: Update BOM
Parts:
- C38, C39: value 4pF -> 4.7pF
- J2, J3, J4: footprint footprints:Jack_3.5mm_PJ-306_Horizontal -> footprints:Jack_3.5mm_PJ-317_Horizontal
Changed lines of the file:
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@@
 			)
 		)
-		(property "Value" "4pF"
+		(property "Value" "4.7pF"
 			(at 0 1.68 90)
 			(layer "F.Fab")
@@
 			)
 		)
-		(property "LCSC" "C1819"
+		(property "LCSC" "C1820"
 			(at 0 0 0)
 			(layer "F.SilkS")
@@
 		)
 	)
-	(footprint "footprints:Jack_3.5mm_PJ-306_Horizontal"
+	(footprint "footprints:Jack_3.5mm_PJ-317_Horizontal"
 		(layer "F.Cu")
 		(at 225.198 97.159 90)
@@
 			)
 		)
-		(property "LCSC" "C692443"
+		(property "LCSC" "C381121"
 			(at 0 0 0)
 			(layer "F.SilkS")
@@
 		(pad "R" thru_hole oval
 			(at -5 -5 90)
-			(size 1.2 2.2)
-			(drill oval 0.4 1.4)
+			(size 1.3 2)
+			(drill oval 0.8 1.5)
 			(layers "*.Cu" "*.Mask")
 			(remove_unused_layers no)
@@
 		(pad "RN" thru_hole oval
 			(at -2.5 -5 90)
-			(size 1.6 2.3)
+			(size 1.3 2)
 			(drill oval 0.8 1.5)
 			(layers "*.Cu" "*.Mask")
@@
 		(pad "S" thru_hole oval
 			(at 0 0 90)
-			(size 2.2 1.2)
-			(drill oval 1.4 0.4)
+			(size 1.3 2)
+			(drill oval 0.8 1.5)
 			(layers "*.Cu" "*.Mask")
 			(remove_unused_layers no)
@@
 		(pad "T" thru_hole oval
 			(at 5 -5 270)
-			(size 1.2 2.2)
-			(drill oval 0.4 1.4)
+			(size 1.3 2)
+			(drill oval 0.8 1.5)
 			(layers "*.Cu" "*.Mask")
 			(remove_unused_layers no)
@@
 		(pad "TN" thru_hole oval
 			(at 2.5 -5 270)
-			(size 1.6 2.5)
+			(size 1.3 2)
 			(drill oval 0.8 1.5)
 			(layers "*.Cu" "*.Mask")
@@
 		)
 		(embedded_fonts no)
-		(model "${KIPRJMOD}/models/AUDIO-TH_PJ-3062-HD-B.step"
+		(model "${KIPRJMOD}/models/AUDIO-TH_3PIN_PJ-317-B.step"
 			(offset
-				(xyz 0 1.5 -4.5)
+				(xyz 0 1 -4)
 			)
 			(scale
@@
 			)
 			(rotate
-				(xyz -0 -0 -90)
+				(xyz -0 -0 -180)
 			)
 		)
@@
 			(pinfunction "PAD")
 			(pintype "passive")
+			(zone_connect 1)
+			(thermal_bridge_width 1)
+			(thermal_bridge_angle 0)
+			(thermal_gap 0.5)
 		)
 		(pad "0" thru_hole circle
@@
 			(pinfunction "PAD")
 			(pintype "passive")
+			(zone_connect 1)
+			(thermal_bridge_width 1)
+			(thermal_bridge_angle 0)
+			(thermal_gap 0.5)
 		)
 		(pad "1" thru_hole roundrect
@@
 			)
 		)
-		(property "Value" "4pF"
+		(property "Value" "4.7pF"
 			(at 0 1.68 90)
 			(layer "F.Fab")
@@
 			)
 		)
-		(property "LCSC" "C1819"
+		(property "LCSC" "C1820"
 			(at 0 0 0)
 			(layer "F.SilkS")
@@
 		)
 	)
-	(footprint "footprints:Jack_3.5mm_PJ-306_Horizontal"
+	(footprint "footprints:Jack_3.5mm_PJ-317_Horizontal"
 		(layer "F.Cu")
 		(at 225.198 84.586 90)
@@
 			)
 		)
-		(property "LCSC" "C692443"
+		(property "LCSC" "C381121"
 			(at 0 0 0)
 			(layer "F.SilkS")
@@
 		(pad "R" thru_hole oval
 			(at -5 -5 90)
-			(size 1.2 2.2)
-			(drill oval 0.4 1.4)
+			(size 1.3 2)
+			(drill oval 0.8 1.5)
 			(layers "*.Cu" "*.Mask")
 			(remove_unused_layers no)
@@
 		(pad "RN" thru_hole oval
 			(at -2.5 -5 90)
-			(size 1.6 2.3)
+			(size 1.3 2)
 			(drill oval 0.8 1.5)
 			(layers "*.Cu" "*.Mask")
@@
 		(pad "S" thru_hole oval
 			(at 0 0 90)
-			(size 2.2 1.2)
-			(drill oval 1.4 0.4)
+			(size 1.3 2)
+			(drill oval 0.8 1.5)
 			(layers "*.Cu" "*.Mask")
 			(remove_unused_layers no)
@@
 		(pad "T" thru_hole oval
 			(at 5 -5 270)
-			(size 1.2 2.2)
-			(drill oval 0.4 1.4)
+			(size 1.3 2)
+			(drill oval 0.8 1.5)
 			(layers "*.Cu" "*.Mask")
 			(remove_unused_layers no)
@@
 		(pad "TN" thru_hole oval
 			(at 2.5 -5 270)
-			(size 1.6 2.5)
+			(size 1.3 2)
 			(drill oval 0.8 1.5)
 			(layers "*.Cu" "*.Mask")
@@
 		)
 		(embedded_fonts no)
-		(model "${KIPRJMOD}/models/AUDIO-TH_PJ-3062-HD-B.step"
+		(model "${KIPRJMOD}/models/AUDIO-TH_3PIN_PJ-317-B.step"
 			(offset
-				(xyz 0 1.5 -4.5)
+				(xyz 0 1 -4)
 			)
 			(scale
@@
 			)
 			(rotate
-				(xyz -0 -0 -90)
+				(xyz -0 -0 -180)
 			)
 		)
@@
 		)
 	)
-	(footprint "footprints:Jack_3.5mm_PJ-306_Horizontal"
+	(footprint "footprints:Jack_3.5mm_PJ-317_Horizontal"
 		(layer "F.Cu")
 		(at 225.198 72.013 90)
@@
 			)
 		)
-		(property "LCSC" "C692443"
+		(property "LCSC" "C381121"
 			(at 0 0 0)
 			(layer "F.SilkS")
@@
 		(pad "R" thru_hole oval
 			(at -5 -5 90)
-			(size 1.2 2.2)
-			(drill oval 0.4 1.4)
+			(size 1.3 2)
+			(drill oval 0.8 1.5)
 			(layers "*.Cu" "*.Mask")
 			(remove_unused_layers no)
@@
 		(pad "RN" thru_hole oval
 			(at -2.5 -5 90)
-			(size 1.6 2.3)
+			(size 1.3 2)
 			(drill oval 0.8 1.5)
 			(layers "*.Cu" "*.Mask")
@@
 		(pad "S" thru_hole oval
 			(at 0 0 90)
-			(size 2.2 1.2)
-			(drill oval 1.4 0.4)
+			(size 1.3 2)
+			(drill oval 0.8 1.5)
 			(layers "*.Cu" "*.Mask")
 			(remove_unused_layers no)
@@
 		(pad "T" thru_hole oval
 			(at 5 -5 270)
-			(size 1.2 2.2)
-			(drill oval 0.4 1.4)
+			(size 1.3 2)
+			(drill oval 0.8 1.5)
 			(layers "*.Cu" "*.Mask")
 			(remove_unused_layers no)
@@
 		(pad "TN" thru_hole oval
 			(at 2.5 -5 270)
-			(size 1.6 2.5)
+			(size 1.3 2)
 			(drill oval 0.8 1.5)
 			(layers "*.Cu" "*.Mask")
@@
 		)
 		(embedded_fonts no)
-		(model "${KIPRJMOD}/models/AUDIO-TH_PJ-3062-HD-B.step"
+		(model "${KIPRJMOD}/models/AUDIO-TH_3PIN_PJ-317-B.step"
 			(offset
-				(xyz 0 1.5 -4.5)
+				(xyz 0 1 -4)
 			)
 			(scale
@@
 			)
 			(rotate
-				(xyz -0 -0 -90)
+				(xyz -0 -0 -180)
 			)
 		)
