File: Audician 32 Plus Replica.kicad_sch (KiCad schematic)
At the start: 67 parts, among them Q1 HT7251, Q2 MMBT3904, U10 74LS138, U6 YMF719E-S, U8 MK1420S, U9 93C66C, X2 33.8688MHz, X3 24.576MHz

Commit message: Add EEPROM with no CDROM
Other:
- note added: "SEL=1, with CD-ROM support: 1-2 10kΩ, 3-4 0Ω, RP1 DNP SEL=2, NO CD-ROM support: 1-3 10kΩ, 2-4 0Ω, RP1 0Ω, U10 DNP"
- note removed: "SEL=1, with CD-ROM support: 1-2 10kΩ, 3-4 0Ω, RP1 DNP SEL=2, NO CD-ROM support: 1-3 10kΩ, 2-4 0Ω, RP1 0Ω"
Changed lines of the file:
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@@
 		(company "Zheng He")
 	)
-	(text "SEL=1, with CD-ROM support:\n1-2 10kΩ, 3-4 0Ω, RP1 DNP\n\nSEL=2, NO CD-ROM support:\n1-3 10kΩ, 2-4 0Ω, RP1 0Ω"
+	(text "SEL=1, with CD-ROM support:\n1-2 10kΩ, 3-4 0Ω, RP1 DNP\n\nSEL=2, NO CD-ROM support:\n1-3 10kΩ, 2-4 0Ω, RP1 0Ω, U10 DNP"
 		(exclude_from_sim no)
 		(at 194.056 113.284 0)

Commit message: Fix BOM Error
Parts:
- CT14: LCSC C112487 -> C2826426
Other:
- note added: "3rd Overtone Replace R29 with 1MΩ if using fundamental crystal"
- note removed: "3rd Overtone"
Changed lines of the file:
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@@
 		)
 	)
-	(text "3rd Overtone"
+	(text "3rd Overtone\nReplace R29 with 1MΩ if using fundamental crystal"
 		(exclude_from_sim no)
-		(at 49.022 112.522 0)
+		(at 49.022 114.554 0)
 		(effects
 			(font
 				(size 1.27 1.27)
 			)
+			(justify left)
 		)
 	)
@@
 			)
 		)
-		(property "LCSC" "C112487"
+		(property "LCSC" "C2826426"
 			(at 35.56 34.29 0)
 			(effects

Commit message: Add notes to schematic
Other:
- note added: "RA2 is populated only when 24MHz crystal is omitted (Not Recommended)"
Changed lines of the file:
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@@
+		)
+	)
+	(text "RA2 is populated only when 24MHz crystal is omitted\n(Not Recommended)"
+		(exclude_from_sim no)
+		(at 63.5 160.274 0)
+		(effects
+			(font
+				(size 1.27 1.27)
+			)
+			(justify left)
 		)
 	)

Commit message: Update BOM
Parts:
- C38, C39: value 22pF -> 4pF; LCSC C1804 -> C1819
- R29: LCSC C17514 -> C17614
Other:
- note added: "3rd Overtone"
- note removed: "3rd Overtone Replace R29 with 1MΩ if using fundamental crystal"
Changed lines of the file:
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@@
 		)
 	)
-	(text "3rd Overtone\nReplace R29 with 1MΩ if using fundamental crystal"
+	(text "3rd Overtone"
 		(exclude_from_sim no)
 		(at 49.022 114.554 0)
@@
 			)
 		)
-		(property "LCSC" "C17514"
+		(property "LCSC" "C17614"
 			(at 36.83 115.57 0)
 			(effects
@@
 			)
 		)
-		(property "Value" "22pF"
+		(property "Value" "4pF"
 			(at 48.768 127 0)
 			(effects
@@
 			)
 		)
-		(property "LCSC" "C1804"
+		(property "LCSC" "C1819"
 			(at 45.72 125.73 0)
 			(effects
@@
 			)
 		)
-		(property "Value" "22pF"
+		(property "Value" "4pF"
 			(at 20.32 127 0)
 			(effects
@@
 			)
 		)
-		(property "LCSC" "C1804"
+		(property "LCSC" "C1819"
 			(at 27.94 125.73 0)
 			(effects

Commit message: Update BOM
Parts:
- C38, C39: value 4pF -> 4.7pF; LCSC C1819 -> C1820
Changed lines of the file:
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@@
 			)
 		)
-		(property "Value" "4pF"
+		(property "Value" "4.7pF"
 			(at 48.768 127 0)
 			(effects
@@
 			)
 		)
-		(property "LCSC" "C1819"
+		(property "LCSC" "C1820"
 			(at 45.72 125.73 0)
 			(effects
@@
 			)
 		)
-		(property "Value" "4pF"
-			(at 20.32 127 0)
+		(property "Value" "4.7pF"
+			(at 19.812 127 0)
 			(effects
 				(font
@@
 			)
 		)
-		(property "LCSC" "C1819"
+		(property "LCSC" "C1820"
 			(at 27.94 125.73 0)
 			(effects
