File: Connectors.kicad_sch (KiCad schematic)
At the start: 59 parts, among them CN1 CD-ROM, J10 Conn_01x04, J11 Conn_01x04, J13 Conn_01x04, J2 Audio Out, J3 Line Input, J4 Microphone, J5 Gameport, J7 Conn_01x04, J8 Conn_01x04, J9 Conn_01x04, U7 Mysterious Chip

Commit message: Fix BOM Error
Parts:
- CT10, CT3: LCSC C160146 -> C106735
Changed lines of the file:
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@@
 			)
 		)
-		(property "LCSC" "C160146"
+		(property "LCSC" "C106735"
 			(at 157.48 63.5 0)
 			(effects
@@
 			)
 		)
-		(property "LCSC" "C160146"
+		(property "LCSC" "C106735"
 			(at 157.48 43.18 0)
 			(effects

Commit message: Update BOM
Parts:
- J2, J3, J4: footprint footprints:Jack_3.5mm_PJ-306_Horizontal -> footprints:Jack_3.5mm_PJ-317_Horizontal; LCSC C692443 -> C381121
Changed lines of the file:
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@@
 			)
 		)
-		(property "Footprint" "footprints:Jack_3.5mm_PJ-306_Horizontal"
+		(property "Footprint" "footprints:Jack_3.5mm_PJ-317_Horizontal"
 			(at 171.45 54.61 0)
 			(effects
@@
 			)
 		)
-		(property "LCSC" "C692443"
+		(property "LCSC" "C381121"
 			(at 171.45 54.61 0)
 			(effects
@@
 			)
 		)
-		(property "Footprint" "footprints:Jack_3.5mm_PJ-306_Horizontal"
+		(property "Footprint" "footprints:Jack_3.5mm_PJ-317_Horizontal"
 			(at 171.45 146.05 0)
 			(effects
@@
 			)
 		)
-		(property "LCSC" "C692443"
+		(property "LCSC" "C381121"
 			(at 171.45 146.05 0)
 			(effects
@@
 			)
 		)
-		(property "Footprint" "footprints:Jack_3.5mm_PJ-306_Horizontal"
+		(property "Footprint" "footprints:Jack_3.5mm_PJ-317_Horizontal"
 			(at 261.62 53.34 0)
 			(effects
@@
 			)
 		)
-		(property "LCSC" "C692443"
+		(property "LCSC" "C381121"
 			(at 261.62 53.34 0)
 			(effects
